File: sch/KiCAD/MultiMeter/MultiMeter.kicad_sch (KiCad schematic)
At the start: 18 parts, among them J1 Conn_01x02_Male, J2 Conn_01x02_Male, J3 Conn_01x03_Male, J4 Conn_01x03_Male, J5 Conn_01x02_Female, J6 Conn_01x15, J7 Conn_01x15

Commit message: 確認用LEDを追加
Parts:
- added D5: (no value), symbol LED:CQY99
- added R5: R, Resistor_THT:R_Axial_DIN0204_L3.6mm_D1.6mm_P7.62mm_Horizontal, symbol Device:R
Connections:
- net at A1.27 (+5V), D2.1 (K), D4.1 (K)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: now also R5.2
- net at A1.29 (GND), A1.4 (GND), C1.2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: now also D5.1 (K)
- new net: D5.2 (A), R5.1
Changed lines of the file:
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@@
   (junction (at 173.99 78.74) (diameter 0) (color 0 0 0 0)
   )
+  (junction (at 64.77 74.93) (diameter 0) (color 0 0 0 0)
+  )
   (junction (at 195.58 44.45) (diameter 0) (color 0 0 0 0)
   )
@@
     (stroke (width 0) (type default) (color 0 0 0 0))
   )
+  (wire (pts (xy 138.43 120.65) (xy 138.43 109.22))
+    (stroke (width 0) (type default) (color 0 0 0 0))
+  )
   (wire (pts (xy 85.09 54.61) (xy 101.6 54.61))
     (stroke (width 0) (type default) (color 0 0 0 0))
@@
     (stroke (width 0) (type default) (color 0 0 0 0))
   )
+  (wire (pts (xy 64.77 74.93) (xy 64.77 120.65))
+    (stroke (width 0) (type default) (color 0 0 0 0))
+  )
   (wire (pts (xy 52.07 62.23) (xy 66.04 62.23))
     (stroke (width 0) (type default) (color 0 0 0 0))
@@
     (stroke (width 0) (type default) (color 0 0 0 0))
   )
+  (wire (pts (xy 125.73 120.65) (xy 138.43 120.65))
+    (stroke (width 0) (type default) (color 0 0 0 0))
+  )
   (wire (pts (xy 90.17 64.77) (xy 90.17 93.98))
     (stroke (width 0) (type default) (color 0 0 0 0))
@@
     (stroke (width 0) (type default) (color 0 0 0 0))
   )
+  (wire (pts (xy 64.77 120.65) (xy 104.14 120.65))
+    (stroke (width 0) (type default) (color 0 0 0 0))
+  )
   (wire (pts (xy 173.99 67.31) (xy 173.99 78.74))
     (stroke (width 0) (type default) (color 0 0 0 0))
@@
   )
   (wire (pts (xy 181.61 20.32) (xy 119.38 20.32))
+    (stroke (width 0) (type default) (color 0 0 0 0))
+  )
+  (wire (pts (xy 111.76 120.65) (xy 118.11 120.65))
     (stroke (width 0) (type default) (color 0 0 0 0))
   )
@@
     (pin "2")
   )
+  (symbol (lib_id "Device:R") (at 107.95 120.65 270) (unit 1)
+    (in_bom yes) (on_board yes)
+    (property "Reference" "R5" (id 0) (at 107.95 118.11 90))
+    (property "Value" "R" (id 1) (at 107.95 120.65 90))
+    (property "Footprint" "Resistor_THT:R_Axial_DIN0204_L3.6mm_D1.6mm_P7.62mm_Horizontal" (id 2) (at 107.95 118.872 90)
+      (effects (font (size 1.27 1.27)) hide)
+    )
+    (property "Datasheet" "~" (id 3) (at 107.95 120.65 0)
+      (effects (font (size 1.27 1.27)) hide)
+    )
+    (pin "1")
+    (pin "2")
+  )
   (symbol (lib_id "Diode:1N4148") (at 43.18 45.72 0) (mirror y) (unit 1)
     (in_bom yes) (on_board yes) (fields_autoplaced)
@@
     )
     (property "Datasheet" "~" (id 3) (at 43.18 55.88 0)
+      (effects (font (size 1.27 1.27)) hide)
+    )
+    (pin "1")
+    (pin "2")
+  )
+  (symbol (lib_id "LED:CQY99") (at 120.65 120.65 0) (mirror y) (unit 1)
+    (in_bom yes) (on_board yes) (fields_autoplaced)
+    (property "Reference" "D5" (id 0) (at 121.793 111.76 0))
+    (property "Value" "" (id 1) (at 121.793 114.3 0))
+    (property "Footprint" "" (id 2) (at 120.65 116.205 0)
+      (effects (font (size 1.27 1.27)) hide)
+    )
+    (property "Datasheet" "https://www.prtice.info/IMG/pdf/CQY99.pdf" (id 3) (at 121.92 120.65 0)
       (effects (font (size 1.27 1.27)) hide)
     )
@@
       (reference "D4") (unit 1) (value "1N4148") (footprint "Diode_THT:D_DO-35_SOD27_P7.62mm_Horizontal")
     )
+    (path "/6d00b441-e462-4628-9c35-00f725ae913f"
+      (reference "D5") (unit 1) (value "CQY99") (footprint "LED_THT:LED_D5.0mm_IRGrey")
+    )
     (path "/e5c8c536-abad-4dbb-a28d-1d01617fbdae"
       (reference "J1") (unit 1) (value "Conn_01x02_Male") (footprint "Connector_Molex:Molex_SPOX_5267-02A_1x02_P2.50mm_Vertical")
@@
       (reference "R4") (unit 1) (value "R") (footprint "Resistor_THT:R_Axial_DIN0204_L3.6mm_D1.6mm_P7.62mm_Horizontal")
     )
-  )
+    (path "/229089b5-d96a-45a7-930c-5b21e68180d7"
+      (reference "R5") (unit 1) (value "R") (footprint "Resistor_THT:R_Axial_DIN0204_L3.6mm_D1.6mm_P7.62mm_Horizontal")
+    )
+  )

Commit message: README.mdを修正
Parts:
- D5: value (none) -> CQY99; footprint (none) -> LED_THT:LED_D5.0mm_IRGrey
Other:
- moved on the sheet: C1
Changed lines of the file:
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@@
     (stroke (width 0) (type default) (color 0 0 0 0))
   )
-  (wire (pts (xy 52.07 20.32) (xy 52.07 45.72))
+  (wire (pts (xy 52.07 25.4) (xy 52.07 45.72))
     (stroke (width 0) (type default) (color 0 0 0 0))
   )
@@
     (stroke (width 0) (type default) (color 0 0 0 0))
   )
-  (wire (pts (xy 33.02 20.32) (xy 13.97 20.32))
+  (wire (pts (xy 33.02 25.4) (xy 13.97 25.4))
     (stroke (width 0) (type default) (color 0 0 0 0))
   )
@@
     (stroke (width 0) (type default) (color 0 0 0 0))
   )
-  (wire (pts (xy 52.07 20.32) (xy 45.72 20.32))
+  (wire (pts (xy 52.07 25.4) (xy 45.72 25.4))
     (stroke (width 0) (type default) (color 0 0 0 0))
   )
@@
     (stroke (width 0) (type default) (color 0 0 0 0))
   )
-  (wire (pts (xy 13.97 20.32) (xy 13.97 45.72))
+  (wire (pts (xy 13.97 25.4) (xy 13.97 45.72))
     (stroke (width 0) (type default) (color 0 0 0 0))
   )
@@
     (in_bom yes) (on_board yes) (fields_autoplaced)
     (property "Reference" "D5" (id 0) (at 121.793 111.76 0))
-    (property "Value" "" (id 1) (at 121.793 114.3 0))
-    (property "Footprint" "" (id 2) (at 120.65 116.205 0)
+    (property "Value" "CQY99" (id 1) (at 121.793 114.3 0))
+    (property "Footprint" "LED_THT:LED_D5.0mm_IRGrey" (id 2) (at 120.65 116.205 0)
       (effects (font (size 1.27 1.27)) hide)
     )
@@
     (pin "2")
   )
-  (symbol (lib_id "pspice:C") (at 39.37 20.32 270) (unit 1)
-    (in_bom yes) (on_board yes) (fields_autoplaced)
-    (property "Reference" "C1" (id 0) (at 39.37 11.43 90))
-    (property "Value" "C" (id 1) (at 39.37 13.97 90))
-    (property "Footprint" "Capacitor_THT:C_Rect_L4.6mm_W2.0mm_P2.50mm_MKS02_FKP02" (id 2) (at 39.37 20.32 0)
-      (effects (font (size 1.27 1.27)) hide)
-    )
-    (property "Datasheet" "~" (id 3) (at 39.37 20.32 0)
-      (effects (font (size 1.27 1.27)) hide)
-    )
+  (symbol (lib_id "pspice:C") (at 39.37 25.4 270) (unit 1)
+    (in_bom yes) (on_board yes) (fields_autoplaced)
+    (property "Reference" "C1" (id 0) (at 39.37 16.51 90))
+    (property "Value" "C" (id 1) (at 39.37 19.05 90))
+    (property "Footprint" "Capacitor_THT:C_Rect_L4.6mm_W2.0mm_P2.50mm_MKS02_FKP02" (id 2) (at 39.37 25.4 0)
+      (effects (font (size 1.27 1.27)) hide)
+    )
+    (property "Datasheet" "~" (id 3) (at 39.37 25.4 0)
+      (effects (font (size 1.27 1.27)) hide)
+    )

Commit message: 微修正
Parts:
- R5: value R -> (none); footprint Resistor_THT:R_Axial_DIN0204_L3.6mm_D1.6mm_P7.62mm_Horizontal -> (none)
Changed lines of the file:
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@@
     (in_bom yes) (on_board yes)
     (property "Reference" "R5" (id 0) (at 107.95 118.11 90))
-    (property "Value" "R" (id 1) (at 107.95 120.65 90))
-    (property "Footprint" "Resistor_THT:R_Axial_DIN0204_L3.6mm_D1.6mm_P7.62mm_Horizontal" (id 2) (at 107.95 118.872 90)
+    (property "Value" "" (id 1) (at 107.95 123.19 90))
+    (property "Footprint" "" (id 2) (at 107.95 118.872 90)
       (effects (font (size 1.27 1.27)) hide)
     )
@@
     )
     (path "/229089b5-d96a-45a7-930c-5b21e68180d7"
-      (reference "R5") (unit 1) (value "R") (footprint "Resistor_THT:R_Axial_DIN0204_L3.6mm_D1.6mm_P7.62mm_Horizontal")
-    )
-  )
+      (reference "R5") (unit 1) (value "200 ohm") (footprint "Resistor_THT:R_Axial_DIN0204_L3.6mm_D1.6mm_P7.62mm_Horizontal")
+    )
+  )

Commit message: 回路図微修正
Parts:
- C1, C2: value C -> (none)
- R1, R2: value R -> 10K ohm
- R3, R4: value R -> (none)
- R5: value (none) -> 200 ohm; footprint (none) -> Resistor_THT:R_Axial_DIN0204_L3.6mm_D1.6mm_P7.62mm_Horizontal
Changed lines of the file:
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@@
     (in_bom yes) (on_board yes)
     (property "Reference" "R4" (id 0) (at 43.18 59.69 90))
-    (property "Value" "R" (id 1) (at 43.18 62.23 90))
+    (property "Value" "" (id 1) (at 46.99 64.77 90))
     (property "Footprint" "Resistor_THT:R_Axial_DIN0204_L3.6mm_D1.6mm_P7.62mm_Horizontal" (id 2) (at 43.18 60.452 90)
       (effects (font (size 1.27 1.27)) hide)
@@
     (in_bom yes) (on_board yes)
     (property "Reference" "R5" (id 0) (at 107.95 118.11 90))
-    (property "Value" "" (id 1) (at 107.95 123.19 90))
-    (property "Footprint" "" (id 2) (at 107.95 118.872 90)
+    (property "Value" "200 ohm" (id 1) (at 107.95 123.19 90))
+    (property "Footprint" "Resistor_THT:R_Axial_DIN0204_L3.6mm_D1.6mm_P7.62mm_Horizontal" (id 2) (at 107.95 118.872 90)
       (effects (font (size 1.27 1.27)) hide)
     )
@@
     (in_bom yes) (on_board yes) (fields_autoplaced)
     (property "Reference" "C2" (id 0) (at 48.26 86.36 90))
-    (property "Value" "C" (id 1) (at 48.26 88.9 90))
+    (property "Value" "" (id 1) (at 48.26 88.9 90))
     (property "Footprint" "Capacitor_THT:C_Rect_L4.6mm_W2.0mm_P2.50mm_MKS02_FKP02" (id 2) (at 48.26 95.25 0)
       (effects (font (size 1.27 1.27)) hide)
@@
     (in_bom yes) (on_board yes)
     (property "Reference" "R3" (id 0) (at 43.18 53.34 90))
-    (property "Value" "R" (id 1) (at 43.18 55.88 90))
+    (property "Value" "" (id 1) (at 50.8 57.15 90))
     (property "Footprint" "Resistor_THT:R_Axial_DIN0204_L3.6mm_D1.6mm_P7.62mm_Horizontal" (id 2) (at 43.18 54.102 90)
       (effects (font (size 1.27 1.27)) hide)
@@
     (in_bom yes) (on_board yes)
     (property "Reference" "R2" (id 0) (at 187.96 57.15 90))
-    (property "Value" "R" (id 1) (at 187.96 59.69 90))
+    (property "Value" "10K ohm" (id 1) (at 195.58 60.96 90))
     (property "Footprint" "Resistor_THT:R_Axial_DIN0204_L3.6mm_D1.6mm_P7.62mm_Horizontal" (id 2) (at 187.96 57.912 90)
       (effects (font (size 1.27 1.27)) hide)
@@
     (in_bom yes) (on_board yes)
     (property "Reference" "R1" (id 0) (at 189.23 45.72 90))
-    (property "Value" "R" (id 1) (at 189.23 48.26 90))
+    (property "Value" "10K ohm" (id 1) (at 196.85 49.53 90))
     (property "Footprint" "Resistor_THT:R_Axial_DIN0204_L3.6mm_D1.6mm_P7.62mm_Horizontal" (id 2) (at 189.23 46.482 90)
       (effects (font (size 1.27 1.27)) hide)
@@
     (in_bom yes) (on_board yes) (fields_autoplaced)
     (property "Reference" "C1" (id 0) (at 39.37 16.51 90))
-    (property "Value" "C" (id 1) (at 39.37 19.05 90))
+    (property "Value" "" (id 1) (at 39.37 19.05 90))
     (property "Footprint" "Capacitor_THT:C_Rect_L4.6mm_W2.0mm_P2.50mm_MKS02_FKP02" (id 2) (at 39.37 25.4 0)
       (effects (font (size 1.27 1.27)) hide)
@@
     )
     (path "/fe839259-c60d-4b91-93e8-3532389c5946"
-      (reference "C1") (unit 1) (value "C") (footprint "Capacitor_THT:C_Rect_L4.6mm_W2.0mm_P2.50mm_MKS02_FKP02")
+      (reference "C1") (unit 1) (value "0.1uF") (footprint "Capacitor_THT:C_Rect_L4.6mm_W2.0mm_P2.50mm_MKS02_FKP02")
     )
     (path "/628b9982-545e-448c-881d-9d848ba0a565"
-      (reference "C2") (unit 1) (value "C") (footprint "Capacitor_THT:C_Rect_L4.6mm_W2.0mm_P2.50mm_MKS02_FKP02")
+      (reference "C2") (unit 1) (value "0.1uF") (footprint "Capacitor_THT:C_Rect_L4.6mm_W2.0mm_P2.50mm_MKS02_FKP02")
     )
     (path "/3ee7be96-43b9-4453-8b59-ad43c1c57ad6"
@@
     )
     (path "/a58d1360-6528-419f-ae62-ad0d63b70a12"
-      (reference "R1") (unit 1) (value "R") (footprint "Resistor_THT:R_Axial_DIN0204_L3.6mm_D1.6mm_P7.62mm_Horizontal")
+      (reference "R1") (unit 1) (value "10K ohm") (footprint "Resistor_THT:R_Axial_DIN0204_L3.6mm_D1.6mm_P7.62mm_Horizontal")
     )
     (path "/a1ab08c6-3248-4afa-9c1c-6e64101b58c1"
-      (reference "R2") (unit 1) (value "R") (footprint "Resistor_THT:R_Axial_DIN0204_L3.6mm_D1.6mm_P7.62mm_Horizontal")
+      (reference "R2") (unit 1) (value "10K ohm") (footprint "Resistor_THT:R_Axial_DIN0204_L3.6mm_D1.6mm_P7.62mm_Horizontal")
     )
     (path "/6a6c5866-364c-4148-b5c1-654fd25e249e"
-      (reference "R3") (unit 1) (value "R") (footprint "Resistor_THT:R_Axial_DIN0204_L3.6mm_D1.6mm_P7.62mm_Horizontal")
+      (reference "R3") (unit 1) (value "10K ohm") (footprint "Resistor_THT:R_Axial_DIN0204_L3.6mm_D1.6mm_P7.62mm_Horizontal")
     )
     (path "/19ba00c8-c3cb-4198-adbb-026273b6dbd1"
-      (reference "R4") (unit 1) (value "R") (footprint "Resistor_THT:R_Axial_DIN0204_L3.6mm_D1.6mm_P7.62mm_Horizontal")
+      (reference "R4") (unit 1) (value "10K ohm") (footprint "Resistor_THT:R_Axial_DIN0204_L3.6mm_D1.6mm_P7.62mm_Horizontal")
     )
     (path "/229089b5-d96a-45a7-930c-5b21e68180d7"

Commit message: 基板修正
Parts:
- removed C1, C2: (no value), Capacitor_THT:C_Rect_L4.6mm_W2.0mm_P2.50mm_MKS02_FKP02, symbol pspice:C
- removed D1, D2, D3, D4: 1N4148, Diode_THT:D_DO-35_SOD27_P7.62mm_Horizontal, symbol Diode:1N4148
- added J8: Conn_01x08_Female, Connector_JST:JST_XH_B8B-XH-A_1x08_P2.50mm_Vertical, symbol Connector:Conn_01x08_Female
- added JP1: Jumper_2_Open, Connector_PinHeader_2.54mm:PinHeader_1x02_P2.54mm_Vertical, symbol Jumper:Jumper_2_Open
- added Q1, Q2: 2SC1815, Package_TO_SOT_THT:TO-92_Inline, symbol Transistor_BJT:2SC1815
- added R10: 7K ohm, Resistor_THT:R_Axial_DIN0204_L3.6mm_D1.6mm_P7.62mm_Horizontal, symbol Device:R
- added R11: 5K ohm, Resistor_THT:R_Axial_DIN0204_L3.6mm_D1.6mm_P7.62mm_Horizontal, symbol Device:R
- added R6, R7, R8, R9: 10K ohm, Resistor_THT:R_Axial_DIN0204_L3.6mm_D1.6mm_P7.62mm_Horizontal, symbol Device:R
- added RV1: RV_Disc_D7mm_W4.5mm_P5mm, Varistor:RV_Disc_D7mm_W4.5mm_P5mm, symbol Device:Varistor
- added TP1, TP2: TestPoint, MountingHole:MountingHole_2.2mm_M2_DIN965_Pad, symbol Connector:TestPoint
- J1, J2: footprint Connector_Molex:Molex_SPOX_5267-02A_1x02_P2.50mm_Vertical -> Connector_Molex:Molex_SPOX_5268-02A_1x02_P2.50mm_Horizontal
- J3, J4: footprint Connector_Molex:Molex_SPOX_5267-03A_1x03_P2.50mm_Vertical -> Connector_Molex:Molex_SPOX_5268-03A_1x03_P2.50mm_Horizontal
- R3, R4: value (none) -> 10K ohm
Connections:
- net at A1.6 (D3), J6.6 (Pin_6): now also R9.1; no longer R4.1
- net +5V: now reaches A1.27 (+5V), J1.1 (Pin_1), J2.1 (Pin_1), J3.1 (Pin_1), J4.1 (Pin_1), J7.12 (Pin_12), R5.2
- net +5V: now also J8.1 (Pin_1), JP1.2 (B), RV1.1
- net at A1.5 (D2), J6.5 (Pin_5): now also R8.1; no longer R3.1
- net GNDPWR: now reaches A1.29 (GND), A1.4 (GND), D5.1 (K), J3.3 (Pin_3), J4.3 (Pin_3), J6.4 (Pin_4), J7.14 (Pin_14), R1.2, R2.2
- net GNDPWR: now also J8.2 (Pin_2), Q1.1 (E), Q2.1 (E), R11.2, RV1.2
- net at A1.23 (A4), J4.2 (Pin_2), J7.8 (Pin_8): now also J8.4 (Pin_4)
- net at A1.24 (A5), J7.9 (Pin_9): now also J8.3 (Pin_3)
- new net: Q2.2 (C), R4.1, R7.1
- new net: R10.1, R11.1, TP1.1
- new net: JP1.1 (A), R6.2, R7.2
- new net: Q1.2 (C), R3.1, R6.1
- new net: Q1.3 (B), R8.2
- new net: Q2.3 (B), R9.2
- new net throttle(+12V - 0V): R10.2, TP2.1
Other:
- moved on the sheet: D5, J5, R3, R4, R5
